Commit message: Replace kinect with d435 in xacro files

File: movo_common/movo_description/urdf/movo.urdf.xacro (robot description, xacro)
@@ -62,5 +62,5 @@
     </gazebo>
     <xacro:movo_base/>
-    <xacro:movo_pan_tilt rgbd_prefix="kinect2" parent="linear_actuator_link">
+    <xacro:movo_pan_tilt rgbd_prefix="d435" parent="linear_actuator_link">
         <origin xyz="0.19735 0 0.3449888" rpy="0 0 0"/>
     </xacro:movo_pan_tilt>

File: movo_common/movo_description/urdf/movo_components/movo_pan_tilt.urdf.xacro (robot description, xacro)
@@ -2,5 +2,5 @@
 <!--
 Software License Agreement (BSD)
-\file      pan_tilt_kinect_one.urdf.xacro
+\file      pan_tilt_d435.urdf.xacro
 \authors   Patrick Hussey
 \copyright Copyright (c) 2017, Kinova Robotics inc. All rights reserved.
@@ -28,5 +28,5 @@
 -->
 <robot name="movo_pan_tilt" xmlns:xacro="http://ros.org/wiki/xacro">
-    <xacro:include filename="$(find movo_description)/urdf/sensors/kinect_one_sensor.urdf.xacro"/>
+    <xacro:include filename="$(find movo_description)/urdf/sensors/_d435.urdf.xacro"/>
     <xacro:property name="M_PI" value="3.14159"/>
     <xacro:macro name="movo_pan_tilt" params="rgbd_prefix parent *origin">
@@ -126,7 +126,7 @@
             </inertial>
 		</link>
-		<xacro:kinect_one_sensor prefix="${rgbd_prefix}" parent="tilt_link">
-			<origin xyz="0.05825 -0.0105875 -0.026" rpy="${-M_PI/2} 0 ${-M_PI/2}" />
-		</xacro:kinect_one_sensor>
+		<xacro:d435_sensor prefix="${rgbd_prefix}" parent="tilt_link">
+			<origin xyz="0 0 0" rpy="${-M_PI/2} 0 ${-M_PI/2}" />
+		</xacro:d435_sensor>
     </xacro:macro>
 </robot>

File: movo_common/movo_description/urdf/pan_tilt_stand_alone.urdf.xacro (robot description, xacro)
@@ -36,5 +36,5 @@
     </gazebo>
     <link name="root"/>
-    <xacro:movo_pan_tilt rgbd_prefix="kinect" parent="root">
+    <xacro:movo_pan_tilt rgbd_prefix="d435" parent="root">
         <origin xyz="0.19735 0 0.3449888" rpy="0 0 0"/>
     </xacro:movo_pan_tilt>
