Commit message: Replace kinect with d435 in xacro files

File: movo_common/movo_description/urdf/movo_components/movo_pan_tilt.urdf.xacro (robot description, xacro)
@@ -126,7 +126,7 @@
             </inertial>
 		</link>
-		<xacro:sensor_d435 parent="tilt_link">
-			<origin xyz="0.06 0 -0.025" rpy="${-M_PI/2} 0 ${-M_PI/2}" />
-		</xacro:sensor_d435>
+		<xacro:d435_sensor prefix="${rgbd_prefix}" parent="tilt_link">
+			<origin xyz="0 0 0" rpy="${-M_PI/2} 0 ${-M_PI/2}" />
+		</xacro:d435_sensor>
     </xacro:macro>
 </robot>

Commit message: Adjust realsense position in urdf

File: movo_common/movo_description/urdf/movo_components/movo_pan_tilt.urdf.xacro (robot description, xacro)
@@ -127,5 +127,5 @@
 		</link>
 		<xacro:sensor_d435 parent="tilt_link">
-			<origin xyz="0 0 0" rpy="${-M_PI/2} 0 ${-M_PI/2}" />
+			<origin xyz="0.06 0 -0.025" rpy="${-M_PI/2} 0 ${-M_PI/2}" />
 		</xacro:sensor_d435>
     </xacro:macro>

Commit message: Flip real sense 180deg around x axis

File: movo_common/movo_description/urdf/movo_components/movo_pan_tilt.urdf.xacro (robot description, xacro)
@@ -127,5 +127,5 @@
 		</link>
 		<xacro:sensor_d435 parent="tilt_link">
-			<origin xyz="0.06 0 -0.025" rpy="${-M_PI/2} 0 ${-M_PI/2}" />
+			<origin xyz="0.08 0 -0.025" rpy="${M_PI/2} 0 ${-M_PI/2}" />
 		</xacro:sensor_d435>
     </xacro:macro>

Commit message: Tilt movo 15 degrees from horizontal

File: movo_common/movo_description/urdf/movo_components/movo_pan_tilt.urdf.xacro (robot description, xacro)
@@ -127,5 +127,5 @@
 		</link>
 		<xacro:sensor_d435 parent="tilt_link">
-			<origin xyz="0.08 0 -0.025" rpy="${M_PI/2} 0 ${-M_PI/2}" />
+			<origin xyz="0.08 0 -0.025" rpy="${M_PI/2} 0 ${-7*M_PI/12}" />
 		</xacro:sensor_d435>
     </xacro:macro>

Commit message: Add tablet box to urdf

File: movo_common/movo_description/urdf/movo_components/movo_pan_tilt.urdf.xacro (robot description, xacro)
@@ -129,4 +129,21 @@
 			<origin xyz="0.08 0 -0.025" rpy="${M_PI/2} 0 ${-7*M_PI/12}" />
 		</xacro:sensor_d435>
+		<joint name="tablet_gimbal" type="fixed">
+			<parent link="tilt_link"/>
+			<child link ="tablet_and_mount"/>
+			<origin xyz="0.07 -0.07 -0.03 " rpy="0 0 ${-M_PI/2}"/>
+		</joint>
+		<link name="tablet_and_mount" parent="tilt_link">
+			<visual>
+			  <geometry>
+			    <box size="0.02 0.24 0.3"/>
+		 	  </geometry>
+			</visual>
+			<collision>
+			  <geometry>
+			    <box size="0.02 0.24 0.3"/>
+		 	  </geometry>
+			</collision>
+		</link>
     </xacro:macro>
 </robot>

Commit message: Add mating block to urdf

File: movo_common/movo_description/urdf/movo_components/movo_pan_tilt.urdf.xacro (robot description, xacro)
@@ -146,4 +146,21 @@
 			</collision>
 		</link>
+		<joint name="mating_gimbal" type="fixed">
+			<parent link="tilt_link"/>
+			<child link ="mating_block"/>
+			<origin xyz="0.09 0 -0.03 " rpy="0 0 0"/>
+		</joint>
+		<link name="mating_block" parent="tilt_link">
+			<visual>
+			  <geometry>
+			    <box size="0.064 0.064 0.11"/>
+		 	  </geometry>
+			</visual>
+			<collision>
+			  <geometry>
+			    <box size="0.064 0.064 0.11"/>
+		 	  </geometry>
+			</collision>
+		</link>
     </xacro:macro>
 </robot>

Commit message: Add camera mount block and move realsense to position

File: movo_common/movo_description/urdf/movo_components/movo_pan_tilt.urdf.xacro (robot description, xacro)
@@ -127,10 +127,10 @@
 		</link>
 		<xacro:sensor_d435 parent="tilt_link">
-			<origin xyz="0.08 0 -0.025" rpy="${M_PI/2} 0 ${-7*M_PI/12}" />
+			<origin xyz="0.22 -0.06 -0.03" rpy="${M_PI/2} 0 ${-7*M_PI/12}" />
 		</xacro:sensor_d435>
 		<joint name="tablet_gimbal" type="fixed">
 			<parent link="tilt_link"/>
 			<child link ="tablet_and_mount"/>
-			<origin xyz="0.07 -0.07 -0.03 " rpy="0 0 ${-M_PI/2}"/>
+			<origin xyz="0.07 -0.06 -0.03 " rpy="0 0 ${-M_PI/2}"/>
 		</joint>
 		<link name="tablet_and_mount" parent="tilt_link">
@@ -163,4 +163,21 @@
 			</collision>
 		</link>
+		<joint name="camera_mount_gimbal" type="fixed">
+			<parent link="tilt_link"/>
+			<child link ="camera_mount"/>
+			<origin xyz="0.15 -0.04 -0.03 " rpy="-${M_PI/2} 0 ${M_PI/2}"/>
+		</joint>
+		<link name="camera_mount" parent="tilt_link">
+			<visual>
+			  <geometry>
+			    <box size="0.01 0.09 0.16"/>
+		 	  </geometry>
+			</visual>
+			<collision>
+			  <geometry>
+			    <box size="0.01 0.09 0.16"/>
+		 	  </geometry>
+			</collision>
+		</link>
     </xacro:macro>
 </robot>

Commit message: Add color and expand collision geometry

File: movo_common/movo_description/urdf/movo_components/movo_pan_tilt.urdf.xacro (robot description, xacro)
@@ -139,8 +139,11 @@
 			    <box size="0.02 0.24 0.3"/>
 		 	  </geometry>
+			  <material name="silver">
+			    <color rgba="0.8 0.8 0.8 1"/>
+		          </material>
 			</visual>
 			<collision>
 			  <geometry>
-			    <box size="0.02 0.24 0.3"/>
+			    <box size="0.04 0.26 0.5"/>
 		 	  </geometry>
 			</collision>
@@ -154,10 +157,11 @@
 			<visual>
 			  <geometry>
-			    <box size="0.064 0.064 0.11"/>
+			    <box size="0.066 0.066 0.13"/>
 		 	  </geometry>
+			  <material name="silver"/>
 			</visual>
 			<collision>
 			  <geometry>
-			    <box size="0.064 0.064 0.11"/>
+			    <box size="0.084 0.084 0.13"/>
 		 	  </geometry>
 			</collision>
@@ -173,8 +177,9 @@
 			    <box size="0.01 0.09 0.16"/>
 		 	  </geometry>
+			  <material name="silver"/>
 			</visual>
 			<collision>
 			  <geometry>
-			    <box size="0.01 0.09 0.16"/>
+			    <box size="0.03 0.11 0.18"/>
 		 	  </geometry>
 			</collision>

Commit message: Flip realsense right side up

File: movo_common/movo_description/urdf/movo_components/movo_pan_tilt.urdf.xacro (robot description, xacro)
@@ -133,5 +133,5 @@
 		</link>
 		<xacro:sensor_d435 parent="tilt_link">
-			<origin xyz="0.22 -0.06 -0.03" rpy="${M_PI/2} 0 ${-7*M_PI/12}" />
+			<origin xyz="0.2 -0.06 -0.03" rpy="${-M_PI/2} 0 ${-7*M_PI/12}" />
 		</xacro:sensor_d435>
 		<joint name="tablet_gimbal" type="fixed">

Commit message: Rotate camera

File: movo_common/movo_description/urdf/movo_components/movo_pan_tilt.urdf.xacro (robot description, xacro)
@@ -127,5 +127,5 @@
 		</link>
 		<xacro:sensor_d435 parent="tilt_link">
-			<origin xyz="0.22 -0.06 -0.03" rpy="${M_PI/2} 0 ${-7*M_PI/12}" />
+			<origin xyz="0.22 -0.06 -0.03" rpy="${-M_PI/2} 0 ${-7*M_PI/12}" />
 		</xacro:sensor_d435>
 		<joint name="tablet_gimbal" type="fixed">

Commit message: Update position of camera in urdf

File: movo_common/movo_description/urdf/movo_components/movo_pan_tilt.urdf.xacro (robot description, xacro)
@@ -133,10 +133,10 @@
 		</link>
 		<xacro:sensor_d435 parent="tilt_link">
-			<origin xyz="0.2 -0.06 -0.03" rpy="${-M_PI/2} 0 ${-7*M_PI/12}" />
+			<origin xyz="0.196 -0.06 -0.03" rpy="${-M_PI/2} 0 ${-7*M_PI/12}" />
 		</xacro:sensor_d435>
 		<joint name="tablet_gimbal" type="fixed">
 			<parent link="tilt_link"/>
 			<child link ="tablet_and_mount"/>
-			<origin xyz="0.07 -0.06 -0.03 " rpy="0 0 ${-M_PI/2}"/>
+			<origin xyz="0.075 -0.06 -0.03 " rpy="0 0 ${-M_PI/2}"/>
 		</joint>
 		<link name="tablet_and_mount" parent="tilt_link">
