Commit message: Add bin but need dimensions and material file

File: movo_common/movo_description/urdf/manipulation/jaco/jaco_7dof.urdf.xacro (robot description, xacro)
@@ -330,4 +330,85 @@
         </joint>
         <link name="${prefix}ee_link"/>
+	<xacro:property name="isright" value="${prefix}"/>
+	<xacro:if value="${isright == 'right_'}">
+		<material name="wood">
+			<texture filename="manipulation/jaco/wood_texture.material"/>
+		</material>
+		<material name="black">
+			<color rgba="0 0 0 1"/>
+		</material>
+		<joint name="${prefix}bin_handle_joint" type="fixed">
+			<parent link="${prefix}ee_link"/>
+			<child link="${prefix}bin_handle"/>
+			<origin xyz="0 0 0" rpy="0 0 0"/>
+		</joint>
+		<joint name="${prefix}bin_joint" type="fixed">
+			<parent link="${prefix}ee_link"/>
+			<child link="${prefix}bin"/>
+			<origin xyz="0 -0.16 0" rpy="0 0 0"/>
+		</joint>
+		<joint name="${prefix}bin_clamp_1_joint" type="fixed">
+			<parent link="${prefix}ee_link"/>
+			<child link="${prefix}bin_clamp_1"/>
+			<origin xyz="0 -0.05 0.1" rpy="0 0 0"/>
+		</joint>
+		<joint name="${prefix}bin_clamp_2_joint" type="fixed">
+			<parent link="${prefix}ee_link"/>
+			<child link="${prefix}bin_clamp_2"/>
+			<origin xyz="0 -0.05 -0.1" rpy="0 0 0"/>
+		</joint>
+		<link name="${prefix}bin_handle" parent="${prefix}ee_fixed_joint">
+			<visual>
+				<geometry>
+					<cylinder length="0.2" radius="0.02"/>
+				</geometry>
+				<material name="black"/>
+			</visual>
+			<collision>
+				<geometry>
+					<cylinder length="0.25" radius="0.03"/>
+				</geometry>
+			</collision>
+		</link>
+		<link name="${prefix}bin" parent="${prefix}ee_fixed_joint">
+			<visual>
+				<geometry>
+					<box size="0.4 0.15 0.2"/>
+				</geometry>
+				<material name="wood"/>
+			</visual>
+			<collision>
+				<geometry>
+					<box size="0.4 0.15 0.2"/>
+				</geometry>
+			</collision>
+		</link>
+		<link name="${prefix}bin_clamp_1" parent="${prefix}ee_fixed_joint">
+			<visual>
+				<geometry>
+					<box size="0.05 0.13 0.01"/>
+				</geometry>
+				<material name="black"/>
+			</visual>
+			<collision>
+				<geometry>
+					<box size="0.05 0.1 0.01"/>
+				</geometry>
+			</collision>
+		</link>
+		<link name="${prefix}bin_clamp_2" parent="${prefix}ee_fixed_joint">
+			<visual>
+				<geometry>
+					<box size="0.05 0.13 0.01"/>
+				</geometry>
+				<material name="black"/>
+			</visual>
+			<collision>
+				<geometry>
+					<box size="0.05 0.1 0.01"/>
+				</geometry>
+			</collision>
+		</link>
+	</xacro:if>
         <xacro:jaco_7dof_arm_transmission prefix="${prefix}" />
   </xacro:macro>

Commit message: Update bin dimensions and add disable some collisions

File: movo_common/movo_description/urdf/manipulation/jaco/jaco_7dof.urdf.xacro (robot description, xacro)
@@ -351,15 +351,15 @@
 			<parent link="${prefix}ee_link"/>
 			<child link="${prefix}bin_clamp_1"/>
-			<origin xyz="0 -0.05 0.1" rpy="0 0 0"/>
+			<origin xyz="0 -0.05 0.101" rpy="0 0 0"/>
 		</joint>
 		<joint name="${prefix}bin_clamp_2_joint" type="fixed">
 			<parent link="${prefix}ee_link"/>
 			<child link="${prefix}bin_clamp_2"/>
-			<origin xyz="0 -0.05 -0.1" rpy="0 0 0"/>
+			<origin xyz="0 -0.05 -0.101" rpy="0 0 0"/>
 		</joint>
 		<link name="${prefix}bin_handle" parent="${prefix}ee_fixed_joint">
 			<visual>
 				<geometry>
-					<cylinder length="0.2" radius="0.02"/>
+					<cylinder length="0.2032" radius="0.024"/>
 				</geometry>
 				<material name="black"/>
@@ -367,5 +367,5 @@
 			<collision>
 				<geometry>
-					<cylinder length="0.25" radius="0.03"/>
+					<cylinder length="0.21" radius="0.03"/>
 				</geometry>
 			</collision>
@@ -374,5 +374,5 @@
 			<visual>
 				<geometry>
-					<box size="0.4 0.15 0.2"/>
+					<box size="0.305 0.1524 0.2032"/>
 				</geometry>
 				<material name="wood"/>
@@ -380,5 +380,5 @@
 			<collision>
 				<geometry>
-					<box size="0.4 0.15 0.2"/>
+					<box size="0.31 0.16 0.21"/>
 				</geometry>
 			</collision>
@@ -387,5 +387,5 @@
 			<visual>
 				<geometry>
-					<box size="0.05 0.13 0.01"/>
+					<box size="0.0635 0.14 0.00635"/>
 				</geometry>
 				<material name="black"/>
@@ -393,5 +393,5 @@
 			<collision>
 				<geometry>
-					<box size="0.05 0.1 0.01"/>
+					<box size="0.07 0.15 0.007"/>
 				</geometry>
 			</collision>
@@ -400,5 +400,5 @@
 			<visual>
 				<geometry>
-					<box size="0.05 0.13 0.01"/>
+					<box size="0.0635 0.14 0.00635"/>
 				</geometry>
 				<material name="black"/>
@@ -406,5 +406,5 @@
 			<collision>
 				<geometry>
-					<box size="0.05 0.1 0.01"/>
+					<box size="0.07 0.15 0.007"/>
 				</geometry>
 			</collision>

Commit message: Add nicer color for box

File: movo_common/movo_description/urdf/manipulation/jaco/jaco_7dof.urdf.xacro (robot description, xacro)
@@ -332,9 +332,9 @@
 	<xacro:property name="isright" value="${prefix}"/>
 	<xacro:if value="${isright == 'right_'}">
-		<material name="wood">
-			<texture filename="manipulation/jaco/wood_texture.material"/>
-		</material>
 		<material name="black">
 			<color rgba="0 0 0 1"/>
+		</material>
+		<material name="brown">
+			<color rgba="${222/255} ${207/255} ${195/255} 1.0"/>
 		</material>
 		<joint name="${prefix}bin_handle_joint" type="fixed">
@@ -376,5 +376,5 @@
 					<box size="0.305 0.1524 0.2032"/>
 				</geometry>
-				<material name="wood"/>
+				<material name="brown"/>
 			</visual>
 			<collision>

Commit message: flip box since two fingers on bottom (#42)

File: movo_common/movo_description/urdf/manipulation/jaco/jaco_7dof.urdf.xacro (robot description, xacro)
@@ -346,15 +346,15 @@
 			<parent link="${prefix}ee_link"/>
 			<child link="${prefix}bin"/>
-			<origin xyz="0 -0.16 0" rpy="0 0 0"/>
+			<origin xyz="0 0.16 0" rpy="0 0 0"/>
 		</joint>
 		<joint name="${prefix}bin_clamp_1_joint" type="fixed">
 			<parent link="${prefix}ee_link"/>
 			<child link="${prefix}bin_clamp_1"/>
-			<origin xyz="0 -0.05 0.101" rpy="0 0 0"/>
+			<origin xyz="0 0.05 0.101" rpy="0 0 0"/>
 		</joint>
 		<joint name="${prefix}bin_clamp_2_joint" type="fixed">
 			<parent link="${prefix}ee_link"/>
 			<child link="${prefix}bin_clamp_2"/>
-			<origin xyz="0 -0.05 -0.101" rpy="0 0 0"/>
+			<origin xyz="0 0.05 -0.101" rpy="0 0 0"/>
 		</joint>
 		<link name="${prefix}bin_handle" parent="${prefix}ee_fixed_joint">
